File: pcb/footctl.kicad_pcb (KiCad board)
At the start: 2 copper layers, 100 x 100 mm, 46 parts, among them J1 Conn_01x10_Female, J10 Conn_01x05_Female, J11 Conn_01x03_Male, J12 Conn_01x03_Male, J2 Conn_01x10_Female, J3 Conn_01x10_Female, J4 Conn_01x10_Female, J5 Conn_01x10_Female, J6 Conn_01x10_Female, J7 Conn_01x10_Female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

Commit message: update pcb
Parts:
- added C10: C, Capacitor_SMD:C_0603_1608Metric, F.Cu at (88.0, 58.0)
- added C11: C, Capacitor_SMD:C_0603_1608Metric, F.Cu at (87.2, 61.2)
- added H1: MountingHole, MountingHole:MountingHole_3.2mm_M3_Pad, F.Cu at (155.8, 58.8)
- added H2: MountingHole, MountingHole:MountingHole_3.2mm_M3_Pad, F.Cu at (93.8, 55.8)
- DS1: footprint Display:WC1602A -> Connector_PinHeader_2.54mm:PinHeader_1x16_P2.54mm_Vertical
- J11: value Conn_01x03_Male -> EXP2; footprint TerminalBlock:TerminalBlock_Altech_AK300-3_P5.00mm -> footctl:NYS126
- J12: value Conn_01x03_Male -> EXP1; footprint TerminalBlock:TerminalBlock_Altech_AK300-3_P5.00mm -> footctl:NYS126
- moved J12 102.5 mm to (144.8, 40.5), turned to 90 degrees
- moved J11 98.3 mm to (123.2, 40.5), turned to 90 degrees
- moved U5 47.5 mm to (89.5, 46.2)
- moved R9 46.0 mm to (88.8, 38.8)
- moved R8 43.6 mm to (88.7, 42.0)
- turned DS1 to 270 degrees
Routing:
- net /EXP2: track 0.00 -> 93.5 mm, vias 0 -> 2
- net /EXP1: track 0.00 -> 71.3 mm, vias 0 -> 2
- net +3V3: track 80.0 -> 135.3 mm, vias 1 -> 2
- net /LCDD7: track 53.6 -> 50.9 mm
- net /LCDD4: track 62.2 -> 59.6 mm
- net /LCDE: track 75.0 -> 72.4 mm
- net /LCDD5: track 58.8 -> 56.2 mm
- net /LCDRW: track 76.6 -> 74.0 mm
- net /LCDRS: track 79.2 -> 76.6 mm
- net /LCDD6: track 56.9 -> 54.4 mm
- net GND: track 24.7 -> 26.6 mm, vias 18 -> 20

Commit message: update pcb
Parts:
- added J13: Conn_01x05_Female, footctl:KCDX-5S-N, F.Cu at (99.8, 42.5)
- J1, J2, J3, J4, J5, J6, J7, J8: footprint Connector_FFC-FPC:Hirose_FH12-10S-0.5SH_1x10-1MP_P0.50mm_Horizontal -> footctl:Hirose_FH12-10S-0.5SH_1x10-1MP_P0.50mm_Horizontal
- moved R8 13.1 mm to (100.5, 47.8)
- moved R9 10.4 mm to (94.0, 47.8), turned to 180 degrees
- moved U5 1.82 mm to (87.8, 46.8)
- moved C4 0.50 mm to (62.0, 68.3)
- moved C6 0.50 mm to (62.0, 74.0)
Routing:
- net /MIDI_TX: track 0.00 -> 54.5 mm
- net +5V: track 111.3 -> 120.2 mm, vias 1 -> 3
- net Net-(J13-Pad4): track 0.00 -> 5.81 mm
- net Net-(R9-Pad2): track 0.00 -> 4.42 mm
- net Net-(J13-Pad5): track 0.00 -> 2.78 mm
- net GND: track 26.6 -> 28.4 mm, vias 20 -> 22

Commit message: updated pcb
Parts:
- moved J6 3.00 mm to (90.0, 77.0)
- moved J7 3.00 mm to (103.0, 77.0)
Routing:
- net /IO2: track 39.1 -> 42.2 mm
- net /IO9: track 32.3 -> 35.3 mm
- net /IO8: track 32.3 -> 35.3 mm
- net /IO6: track 41.3 -> 44.3 mm
- net /IO5: track 41.5 -> 44.5 mm
- net /IO4: track 41.4 -> 44.4 mm
- net /IO3: track 39.6 -> 42.6 mm
- net /IO10: track 32.4 -> 35.4 mm
- net /IO0: track 37.9 -> 40.9 mm
- net /IO7: track 41.3 -> 44.3 mm
- net /IO11: track 32.3 -> 35.3 mm
- net /IO1: track 38.5 -> 41.5 mm
